File: Hardware/DC34_Cnet_Badge_Main/DC34_Cnet_Badge_Main.kicad_pcb (KiCad board)
At the start: 2 copper layers, 220.5 x 272.8 mm, 9 parts, among them J1 LCD_Display, J2 Micro_SDCard, J3 RFID-RC522, J4 JST_PH_S2B-PH-K_1x02_P2.00mm_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, J5 SAO, U1 MH-CD42_LiPo_Batery_Managemen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

Commit message: klip-updates
klip-updates
Parts:
- moved U1 175.5 mm to (137.7, 203.1)
- moved J4 156.0 mm to (139.4, 159.2), turned to 180 degrees
- moved D1 88.5 mm to (60.0, 160.7)
- moved S1 66.4 mm to (15.3, 6.99), turned to -153 degrees
