File: Hardware/DC34_Cnet_Badge_Main/DC34_Cnet_Badge_Main.kicad_pcb (KiCad board)
At the start: 2 copper layers, 3.6 x 7 mm, 8 parts, among them J1 LCD_Display, J2 Micro_SDCard, J3 RFID-RC522, J4 JST_PH_S2B-PH-K_1x02_P2.00mm_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, J5 SAO, U1 MH-CD42_LiPo_Batery_Managemen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

Commit message: Updates
Parts:
- J2, J3, J4, U1, U2: moved to B.Cu
- moved J4 332.7 mm to (217.0, 147.0), turned to 180 degrees
- moved J5 303.1 mm to (108.2, -44.8), turned to 135 degrees
- moved U2 268.7 mm to (207.0, 84.5), turned to -90 degrees
- moved S1 257.6 mm to (241.4, 142.5)
- moved J1 236.8 mm to (148.0, 13.5)
- moved J2 201.2 mm to (152.3, -62.3), turned to 180 degrees
- moved J3 194.8 mm to (152.8, 154.7), turned to -105 degrees
- moved U1 130.1 mm to (174.2, 224.7), turned to 180 degrees
Other:
- board size 3.6 x 7 mm -> 199.9 x 329.4 mm

Commit message: PCB Updates
Parts:
- added D1: LED, LED_THT:LED_D3.0mm, F.Cu at (53.5, 60.5)
- added Ref**: Val**, DC34_Cnet_Badge_Main:CompuNet PCB Logo, B.Cu at (38.0, 36.5)
- U2: moved to F.Cu
- moved J2 103.3 mm to (80.5, 12.0)
- moved U2 96.8 mm to (120.5, 41.0), turned to 180 degrees
- moved S1 95.1 mm to (146.5, 148.5), turned to 180 degrees
- moved J1 93.1 mm to (57.0, 33.0), turned to 90 degrees
- moved J3 92.4 mm to (66.0, 123.0), turned to -90 degrees
- moved J4 84.2 mm to (133.0, 153.4), turned to 0 degrees
- moved U1 60.0 mm to (145.7, 171.8), turned to 0 degrees
- moved J5 51.9 mm to (104.5, 7.00), turned to 90 degrees
Routing:
- net Net-(J1-SCL): track 0.00 -> 171.5 mm, vias 0 -> 1
- net Net-(J1-SDA): track 0.00 -> 155.1 mm
- net Net-(J2-MISO): track 0.00 -> 148.3 mm, vias 0 -> 1
- net Net-(J3-RST): track 0.00 -> 113.9 mm
- net Net-(J1-RST): track 0.00 -> 112.7 mm, vias 0 -> 1
- net Net-(J2-CS): track 0.00 -> 108.6 mm, vias 0 -> 1
- net Net-(J3-SDA): track 0.00 -> 104.1 mm, vias 0 -> 2
- net Net-(J1-CS): track 0.00 -> 73.1 mm
- net Net-(J1-DC): track 0.00 -> 72.7 mm
- net Net-(J5-Pin_5): track 0.00 -> 53.0 mm
- net Net-(J5-Pin_6): track 0.00 -> 50.6 mm
- net Net-(U1-VIN): track 0.00 -> 28.0 mm
- net Net-(J4-Pin_1): track 0.00 -> 17.2 mm
- net Net-(U1-OUT): track 0.00 -> 9.76 mm
- net GND: track 0.00 -> 8.50 mm, vias 0 -> 2
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- added copper zone on F.Cu, net +3V3
- added copper zone on B.Cu, net GND
Other:
- board size 199.9 x 329.4 mm -> 150 x 175 mm
- board text added: "@slash128v6 https://github.com/slash128v6/DC34_Cnet_Badge"
- board text added: "LIPO"
- board text added: "MALWARE SCAN TOOL 3000 (MST3K)"

Commit message: Incremental updates
Other:
- board text added: "*"

Commit message: Alternate Layout
Alternate Layout
Parts:
- removed Ref**: Val**, DC34_Cnet_Badge_Main:CompuNet PCB Logo
- U2: moved to B.Cu
- moved U2 160.8 mm to (177.1, 191.5), turned to 90 degrees
- moved S1 145.1 mm to (12.1, 203.1)
- moved J5 127.5 mm to (23.5, 105.5)
- moved J3 94.3 mm to (160.3, 121.8)
- moved J2 89.8 mm to (4.63, -36.0), turned to -45 degrees
- moved J4 53.8 mm to (118.6, 205.3), turned to 90 degrees
- moved U1 32.6 mm to (124.9, 196.9), turned to 180 degrees
- moved J1 19.3 mm to (49.5, 15.2), turned to 0 degrees
- moved D1 15.4 mm to (58.9, 74.9), turned to 0 degrees
Routing:
- net Net-(J1-SCL): track 171.5 -> 5.54 mm, vias 1 -> 0
- net Net-(J1-SDA): track 155.1 -> 0.00 mm
- net Net-(J2-MISO): track 148.3 -> 0.00 mm, vias 1 -> 0
- net Net-(J3-RST): track 113.9 -> 0.00 mm
- net Net-(J1-RST): track 112.7 -> 0.00 mm, vias 1 -> 0
- net Net-(U1-OUT): track 9.76 -> 119.9 mm
- net Net-(J2-CS): track 108.6 -> 0.00 mm, vias 1 -> 0
- net Net-(J3-SDA): track 104.1 -> 0.00 mm, vias 2 -> 0
- net Net-(U1-VIN): track 28.0 -> 118.7 mm
- net Net-(J1-CS): track 73.1 -> 0.00 mm
- net Net-(J1-DC): track 72.7 -> 0.00 mm
- net Net-(J5-Pin_5): track 53.0 -> 0.00 mm
- net Net-(J5-Pin_6): track 50.6 -> 0.00 mm
- net GND: track 8.50 -> 23.4 mm, vias 2 -> 0
- net Net-(J4-Pin_1): track 17.2 -> 6.70 mm
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- removed copper zone on F.Cu, net +3V3
- removed copper zone on B.Cu, net GND
Other:
- board size 150 x 175 mm -> 220.5 x 269.4 mm
- board text removed: "*"

Commit message: Version 2
Version 2 Layout
Parts:
- moved S1 207.5 mm to (81.7, 7.56)
- moved J4 183.9 mm to (40.0, 39.0)
- moved U1 164.6 mm to (60.8, 45.3), turned to -90 degrees
- moved U2 85.8 mm to (123.6, 124.5)
- moved J3 75.0 mm to (85.4, 118.0)
- moved J2 14.3 mm to (-7.64, -43.3), turned to -136 degrees
- moved J5 13.0 mm to (11.0, 101.9)
- moved D1 10.9 mm to (48.2, 73.1)
- moved J1 9.56 mm to (40.4, 12.6)
Routing:
- net Net-(U1-OUT): track 119.9 -> 0.00 mm
- net Net-(U1-VIN): track 118.7 -> 0.00 mm
- net GND: track 23.4 -> 0.00 mm
- net Net-(J4-Pin_1): track 6.70 -> 0.00 mm
- net Net-(J1-SCL): track 5.54 -> 0.00 mm
- net +3V3: track 3.20 -> 0.00 mm
Other:
- board size 220.5 x 269.4 mm -> 220.5 x 272.8 mm

Commit message: Traces run
Parts:
- added Ref**: Val**, DC34_Cnet_Badge_Main:CompuNet PCB Logo, F.Cu at (26.5, 191.0)
- added Ref**: Val**, DC34_Cnet_Badge_Main:CompuNet PCB Logo, B.Cu at (27.5, 191.0)
- S1: moved to B.Cu
- moved J4 182.0 mm to (140.0, 191.0)
- moved U1 163.9 mm to (156.8, 178.2), turned to 180 degrees
- moved J5 151.2 mm to (160.9, 81.9), turned to 45 degrees
- moved S1 85.2 mm to (9.14, -37.2), turned to 48 degrees
- moved D1 42.9 mm to (18.0, 103.5)
- moved U2 15.5 mm to (138.8, 127.9)
- moved J1 12.8 mm to (47.0, 23.5)
- moved J3 1.69 mm to (87.0, 117.5)
Routing:
- net Net-(J1-SCL): track 0.00 -> 328.6 mm
- net Net-(U1-OUT): track 0.00 -> 328.4 mm
- net Net-(U1-VIN): track 0.00 -> 318.3 mm
- net Net-(J1-SDA): track 0.00 -> 310.4 mm, vias 0 -> 2
- net Net-(J2-CS): track 0.00 -> 303.9 mm
- net Net-(J2-MISO): track 0.00 -> 298.3 mm
- net Net-(J1-RST): track 0.00 -> 257.3 mm
- net Net-(J1-DC): track 0.00 -> 228.8 mm
- net Net-(J1-CS): track 0.00 -> 202.0 mm
- net +3V3: track 0.00 -> 193.1 mm, vias 0 -> 2
- net GND: track 0.00 -> 98.2 mm
- net Net-(J5-Pin_6): track 0.00 -> 59.6 mm
- net Net-(J3-RST): track 0.00 -> 59.2 mm
- net Net-(J5-Pin_5): track 0.00 -> 47.8 mm
- net Net-(J3-SDA): track 0.00 -> 35.3 mm
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- added copper zone on F.Cu, net +3V3
- added copper zone on B.Cu, net GND
Other:
- outline, holes or cut-outs redrawn
